File: pro_fdd_drive_upper_pcb/x68_pro_fdd_eject_drive_board.sch (KiCad schematic (older format))
At the start: 23 parts, among them J51 CONN_01x06, J53 CONN_01x16, J54 DISK_PRESENT_SENSOR, M1 Motor_DC_ALT, U51 74HC14, U52 LB1460

Commit message: Add files via upload
Other:
- note added: "IC215-pin11 (74LS541)"
- note added: "IC215-pin12 (74LS541)"
- note added: "IC215-pin13 (74LS541)"
- note added: "IC215-pin16 (74LS541)"
- note added: "IC215-pin17 (74LS541)"
- note added: "IC215-pin18 (74LS541)"
- note added: "OUTPUT from IC215 (74LS541) -pin11"
- note added: "to IC217-pin11 (74LS07), input"
- note added: "to IC217-pin13 (74LS07), input"
- note added: "to IC217-pin5 (74LS07), input"
- note added: "to IC217-pin9 (74LS07), input"
- note added: "to IX1269C-39, input"
Changed lines of the file:
@@
 Text GLabel 5650 6600 0    50   Input ~ 0
 DISKONBACK
+Text Notes 3950 3400 0    50   ~ 0
+OUTPUT from IC215 (74LS541) -pin11
+Text Notes 4350 6250 0    50   ~ 0
+IC215-pin18 (74LS541)
+Text Notes 3850 6350 0    50   ~ 0
+to IC217-pin13 (74LS07), input
+Text Notes 4350 6450 0    50   ~ 0
+IC215-pin17 (74LS541)
+Text Notes 4350 6550 0    50   ~ 0
+IC215-pin16 (74LS541)
+Text Notes 3800 6850 0    50   ~ 0
+to IC217-pin5 (74LS07), input
+Text Notes 3850 6750 0    50   ~ 0
+to IC217-pin11 (74LS07), input
+Text Notes 4050 7150 0    50   ~ 0
+to IC217-pin9 (74LS07), input
+Text Notes 4000 7350 0    50   ~ 0
+to IX1269C-39, input
+Text Notes 4350 7050 0    50   ~ 0
+IC215-pin13 (74LS541)
+Text Notes 4350 7250 0    50   ~ 0
+IC215-pin12 (74LS541)
+Text Notes 4100 7450 0    50   ~ 0
+IC215-pin11 (74LS541)
 $EndSCHEMATC
